Commit message: working multi DOF am

File: models/aerialmanipulator.urdf (robot description, URDF)
Before this commit: robot AerialManipulator, 12 links, 11 joints
Joints:
- joint joint2: type continuous -> fixed
- joint prop1: axis (none) -> 0 0 1; type fixed -> continuous
- joint prop2: axis (none) -> 0 0 1; type fixed -> continuous
- joint prop3: axis (none) -> 0 0 1; type fixed -> continuous
- joint prop4: axis (none) -> 0 0 1; type fixed -> continuous
