Commit message: Ball Catching Env working prototype

File: models/aerial_manipulator_debug.urdf (robot description, URDF)
Before this commit: robot AerialManipulator, 10 links, 9 joints
Links:
- added link link1, mass 0.053412; visual box size=.009 .004 .041; visual cylinder length=0.022 radius=.0142
- added link link2, mass 0.07583633; visual box size=.004 .022 .03; visual box size=.004 .022 .03
- added link virtualvehicle, mass 0.0000000000001; visual box size=.009 .0455 .004; visual box size=.036 .071 .022
- link endeffector: mass 0.1 -> None
- link vehicle: geometry 
Joints:
- added joint joint1: type fixed, parent link1, child virtualvehicle, origin xyz=0 0 -.1607 rpy=0 1.57079632679 0, axis 0 1 0, limit lower=-3.0 upper=3.0 effort=.9 velocity=1e9
- added joint joint2: type fixed, parent link2, child link1, origin xyz= 0 0 -.0625 rpy=0 0 -1.57079632679, axis 0 0 1, limit lower=-3.1415926 upper=3.1415926 effort=.1 velocity=1e9
- added joint yawfix: type fixed, parent virtualvehicle, child vehicle, origin xyz=0 0 0 rpy=0 0 1.57079632679
- joint jointend: child vehicle -> link2; origin xyz=-0.2 0 0 rpy=0 0 0 -> xyz=0 0 0 rpy=-1.57079632679 0 0
