Commit message: working SE(3) baseline)

File: models/aerial_manipulator_0dof_debug.urdf (robot description, URDF)
Before this commit: robot AerialManipulator, 12 links, 11 joints
Links:
- added link virtualvehicle, mass 0.0000000000001; visual box size=.009 .0455 .004; visual box size=.036 .071 .022
- link vehicle: mass 0.706028 -> 0.83527633; geometry 
Joints:
- added joint yawfix: type fixed, parent virtualvehicle, child vehicle, origin xyz=0 0 0 rpy=0 0 1.57079632679
- joint joint1: child vehicle -> virtualvehicle

Commit message: updating models

File: models/aerial_manipulator_0dof_debug.urdf (robot description, URDF)
Before this commit: robot AerialManipulator, 13 links, 12 joints
Links:
- link link1: mass 0.0000000000001 -> None
- link link2: mass 0.0000000000001 -> None
- link virtualvehicle: mass 0.0000000000001 -> None
Joints:
- joint jointend: origin xyz=0 0 0 rpy=-1.57 0 0 -> xyz=0 0 0 rpy=-1.57079632679 0 0

File: models/aerial_manipulator_0dof_orig.urdf (robot description, URDF)
Before this commit: robot AerialManipulator, 13 links, 12 joints
Links:
- removed link virtualvehicle
- link link1: mass None -> .053412
- link link2: mass None -> 0.07583633
- link vehicle: mass 0.83527633 -> 0.706028; geometry visual box size=.009 .0455 .004; visual box size=.036 .071 .022
Joints:
- removed joint yawfix
- joint joint1: child virtualvehicle -> vehicle
- joint jointend: origin xyz=0 0 0 rpy=-1.57079632679 0 0 -> xyz=0 0 0 rpy=-1.57 0 0
