Commit message: Update after ICRA

File: models/aerial_manipulator_0dof_debug_catching.urdf (robot description, URDF)
Before this commit: robot AerialManipulator, 13 links, 12 joints
Links:
- link link1: mass 0.0000000000001 -> None
- link link2: mass 0.0000000000001 -> None
- link virtualvehicle: mass 0.0000000000001 -> None
Joints:
- joint jointend: origin xyz=0 0 0 rpy=-1.57 0 0 -> xyz=0 0 0 rpy=-1.57079632679 0 0

File: models/aerial_manipulator_1dof_wrist.urdf (robot description, URDF)
Before this commit: robot AerialManipulator, 13 links, 12 joints
Links:
- removed link virtualvehicle
- link endeffector: geometry 
- link link1: mass None -> .053412
- link link2: mass None -> 0.07583633
- link vehicle: mass 0.83527633 -> 0.706028; geometry visual box size=.009 .0455 .004; visual box size=.036 .071 .022
Joints:
- removed joint yawfix
- joint joint1: child virtualvehicle -> vehicle
- joint joint2: type fixed -> continuous
- joint jointend: origin xyz=0 0 0 rpy=-1.57079632679 0 0 -> xyz=0 0 0 rpy=-1.57 0 0
