Commit message: updating models

File: models/aerial_manipulator_0dof.urdf (robot description, URDF)
Before this commit: robot AerialManipulator, 13 links, 12 joints
Links:
- added link COM
Joints:
- added joint com_offset: type fixed, parent endeffector, child COM, origin xyz=0 -2.00715814e-01 -1.59835415e-04 rpy=0 0 0

File: models/aerial_manipulator_0dof_debug_working_pinocchio.urdf (robot description, URDF)
Before this commit: robot AerialManipulator, 7 links, 6 joints
Links:
- link endeffector: mass None -> 0.2
Joints:
- joint prop1: type continuous -> fixed
- joint prop2: type continuous -> fixed
- joint prop3: type continuous -> fixed
- joint prop4: type continuous -> fixed

File: models/aerial_manipulator_1dof.urdf (robot description, URDF)
Before this commit: robot AerialManipulator, 12 links, 11 joints
Links:
- added link COM
- added link virtualvehicle; visual box size=.009 .0455 .004; visual box size=.036 .071 .022
- link vehicle: mass 0.706028 -> 0.83527633; geometry 
Joints:
- added joint com_offset: type fixed, parent endeffector, child COM, origin xyz=0 -2.00715814e-01 -1.59835415e-04 rpy=0 0 0
- added joint yawfix: type fixed, parent virtualvehicle, child vehicle, origin xyz=0 0 0 rpy=0 0 1.57079632679
