Commit message: Updating environments for cross-evaluations.

File: models/aerial_manipulator_0dof_debug_working.urdf (robot description, URDF)
Before this commit: robot AerialManipulator, 7 links, 6 joints
Links:
- added link gripper; visual box size=.004 .022 .03; visual box size=.004 .022 .03

File: models/uam_0dof_long_arm_com_middle.urdf (robot description, URDF)
Before this commit: robot AerialManipulator, 14 links, 13 joints
Links:
- link arm: geometry visual cylinder length=0.022 radius=.0142; visual cylinder length=0.31499999999999995 radius=.0075
Joints:
- joint com_placement: origin xyz=0 -0.2 0 rpy=0 0 0 -> xyz=0 -0.36 0 rpy=0 0 0
- joint vehicle_attachment: origin xyz=0 0 -0.15 rpy=1.57079632679 1.57079632679 0 -> xyz=0 0 -0.35 rpy=1.57079632679 1.57079632679 0
