Commit message: rss submission upload

File: models/uam_0dof_catching.urdf (robot description, URDF)
Before this commit: robot AerialManipulator, 14 links, 13 joints
Links:
- link arm: geometry visual cylinder length=0.022 radius=.0142; visual cylinder length=0.11499999999999999 radius=.0075
- link endeffector: geometry collision cylinder length=.02 radius=.04; visual cylinder length=.02 radius=.04
